Commit message: Updated zu5 URDF and meshes

File: src/jaka_description/urdf/jaka_zu5.urdf (robot description, URDF)
Before this commit: robot jaka_zu5, 8 links, 7 joints
Links:
- removed link Link_0
- removed link Link_1
- removed link Link_2
- removed link Link_3
- removed link Link_4
- removed link Link_5
- removed link Link_6
- added link Link1, mass 2.877; collision mesh filename=package://jaka_description/meshes/jaka_zu5_meshes/Link1.STL; visual mesh filename=package://jaka_description/meshes/jaka_zu5_meshes/Link1.STL
- added link Link2, mass 7.293; collision mesh filename=package://jaka_description/meshes/jaka_zu5_meshes/Link2.STL; visual mesh filename=package://jaka_description/meshes/jaka_zu5_meshes/Link2.STL
- added link Link3, mass 1.707; collision mesh filename=package://jaka_description/meshes/jaka_zu5_meshes/Link3.STL; visual mesh filename=package://jaka_description/meshes/jaka_zu5_meshes/Link3.STL
- added link Link4, mass 1.184; collision mesh filename=package://jaka_description/meshes/jaka_zu5_meshes/Link4.STL; visual mesh filename=package://jaka_description/meshes/jaka_zu5_meshes/Link4.STL
- added link Link5, mass 1.228; collision mesh filename=package://jaka_description/meshes/jaka_zu5_meshes/Link5.STL; visual mesh filename=package://jaka_description/meshes/jaka_zu5_meshes/Link5.STL
- added link Link6, mass 0.289; collision mesh filename=package://jaka_description/meshes/jaka_zu5_meshes/Link6.STL; visual mesh filename=package://jaka_description/meshes/jaka_zu5_meshes/Link6.STL
- added link link0, mass 0.905; collision mesh filename=package://jaka_description/meshes/jaka_zu5_meshes/link0.STL; visual mesh filename=package://jaka_description/meshes/jaka_zu5_meshes/link0.STL
Joints:
- joint fixed: child Link_0 -> link0
- joint joint_1: child Link_1 -> Link1; origin xyz=0 0 0.12015 rpy=0 0 0 -> xyz=0 -0.00022535 0.12015 rpy=0 0 0; parent Link_0 -> link0
- joint joint_2: child Link_2 -> Link2; parent Link_1 -> Link1
- joint joint_3: child Link_3 -> Link3; parent Link_2 -> Link2
- joint joint_4: child Link_4 -> Link4; parent Link_3 -> Link3
- joint joint_5: child Link_5 -> Link5; parent Link_4 -> Link4
- joint joint_6: child Link_6 -> Link6; parent Link_5 -> Link5
